Commit message: fix(description): 多ロボット(dual-arm)対応 — material prefix化と GPIO生成条件の統一
同一 URDF に複数 RV-2FR を prefix 付きで載せる際の不整合を修正。

- 全モデルの <material name="white"> 等を ${prefix} 付きに変更し、複数台搭載時の
  material 名衝突を回避(prefix="" では従来どおり "white" となり後方互換)。
- rv2fr.hardware.xacro: GPIO 生成条件が $(arg use_fake_hardware)(グローバル arg)を
  見ており、関節 hardware の ${use_fake_hardware}(マクロ param)と不整合だった。
  param 参照へ統一し、結合ロボットで per-arm に実機/sim を混在させても実機側に
  GPIO が生成されるようにした。これがないと実機側が
  "0 GPIO components, 5 expected" で初期化失敗する(単腕は arg==param で不変)。

File: melfa_description/ros2_control/rv2fr.hardware.xacro (robot description, xacro)
@@ -141,5 +141,5 @@
             </gpio>
             </xacro:macro>
-            <xacro:unless value="$(arg use_fake_hardware)">
+            <xacro:unless value="${use_fake_hardware}">
                 <xacro:if value="${controller_type == 'R'}">
                     <!-- R Type Controller IO -->

File: melfa_description/urdf/rh6crh6020/rh6crh6020_macro.xacro (robot description, xacro)
@@ -19,5 +19,5 @@
         <xacro:property name="wrist_mass" value="0.12190" />
         <xacro:property name="hand_flange_mass" value="0.01879" />
-        <material name="white">
+        <material name="${prefix}white">
             <color rgba="1.0 1.0 1.0 1.0"/>
         </material>
@@ -68,5 +68,5 @@
         <link name="${prefix}rh6crh6020_base">
             <visual>
-                <material name="white"/>
+                <material name="${prefix}white"/>
                 <origin rpy="0 0 0" xyz="0 0 0"/>
                 <geometry>
@@ -86,5 +86,5 @@
         <link name="${prefix}rh6crh6020_no1arm">
             <visual>
-                <material name="white"/>
+                <material name="${prefix}white"/>
                 <origin rpy="0 0 0" xyz="0 0 0"/>
                 <geometry>
@@ -104,5 +104,5 @@
         <link name="${prefix}rh6crh6020_no2arm">
             <visual>
-            <material name="white"/>
+            <material name="${prefix}white"/>
             <origin rpy="0 0 0" xyz="0 0 0"/>
             <geometry>
@@ -127,5 +127,5 @@
         <link name="${prefix}rh6crh6020_shaft">
             <visual>
-                <material name="white"/>
+                <material name="${prefix}white"/>
                 <origin rpy="0 0 0" xyz="0 0 0"/>
                 <geometry>

File: melfa_description/urdf/rh6frh5520/rh6frh5520_macro.xacro (robot description, xacro)
@@ -19,5 +19,5 @@
         <xacro:property name="wrist_mass" value="0.12190" />
         <xacro:property name="hand_flange_mass" value="0.01879" />
-        <material name="white">
+        <material name="${prefix}white">
             <color rgba="1.0 1.0 1.0 1.0"/>
         </material>
@@ -68,5 +68,5 @@
         <link name="${prefix}rh6frh5520_base">
             <visual>
-                <material name="white"/>
+                <material name="${prefix}white"/>
                 <origin rpy="0 0 0" xyz="0 0 0"/>
                 <geometry>
@@ -86,5 +86,5 @@
         <link name="${prefix}rh6frh5520_no1arm">
             <visual>
-                <material name="white"/>
+                <material name="${prefix}white"/>
                 <origin rpy="0 0 0" xyz="0 0 0"/>
                 <geometry>
@@ -104,5 +104,5 @@
         <link name="${prefix}rh6frh5520_no2arm">
             <visual>
-                <material name="white"/>
+                <material name="${prefix}white"/>
                 <origin rpy="0 0 0" xyz="0 0 0"/>
                 <geometry>
@@ -127,5 +127,5 @@
         <link name="${prefix}rh6frh5520_shaft">
             <visual>
-                <material name="white"/>
+                <material name="${prefix}white"/>
                 <origin rpy="0 0 0" xyz="0 0 0"/>
                 <geometry>

File: melfa_description/urdf/rv13frl/rv13frl_macro.xacro (robot description, xacro)
@@ -19,5 +19,5 @@
         <xacro:property name="wrist_mass" value="0.12190" />
         <xacro:property name="hand_flange_mass" value="0.01879" />
-        <material name="white">
+        <material name="${prefix}white">
             <color rgba="1.0 1.0 1.0 1.0"/>
         </material>
@@ -84,5 +84,5 @@
         <link name="${prefix}rv13frl_base">
             <visual>
-            <material name="white"/>
+            <material name="${prefix}white"/>
             <origin rpy="0 0 0" xyz="0 0 0"/>
             <geometry>
@@ -102,5 +102,5 @@
         <link name="${prefix}rv13frl_shoulder">
             <visual>
-            <material name="white"/>
+            <material name="${prefix}white"/>
             <origin rpy="0 0 0" xyz="0 0 0"/>
             <geometry>
@@ -120,5 +120,5 @@
         <link name="${prefix}rv13frl_upper_arm">
             <visual>
-            <material name="white"/>
+            <material name="${prefix}white"/>
             <origin rpy="0 0 0" xyz="0 0 0"/>
             <geometry>
@@ -138,5 +138,5 @@
         <link name="${prefix}rv13frl_elbow">
             <visual>
-            <material name="white"/>
+            <material name="${prefix}white"/>
             <origin rpy="0 0 0" xyz="0 0 0"/>
             <geometry>
@@ -156,5 +156,5 @@
         <link name="${prefix}rv13frl_forearm">
             <visual>
-            <material name="white"/>
+            <material name="${prefix}white"/>
             <origin rpy="0 0 0" xyz="0 0 0"/>
             <geometry>
@@ -174,5 +174,5 @@
         <link name="${prefix}rv13frl_wrist">
             <visual>
-            <material name="white"/>
+            <material name="${prefix}white"/>
             <origin rpy="0 0 0" xyz="0 0 0"/>
             <geometry>
@@ -192,5 +192,5 @@
         <link name="${prefix}rv13frl_hand_flange">
             <visual>
-            <material name="white"/>
+            <material name="${prefix}white"/>
             <origin rpy="0 0 0" xyz="0 0 0"/>
             <geometry>

File: melfa_description/urdf/rv2fr/rv2fr_macro.xacro (robot description, xacro)
@@ -19,5 +19,5 @@
         <xacro:property name="wrist_mass" value="0.12190" />
         <xacro:property name="hand_flange_mass" value="0.12190" />
-        <material name="white">
+        <material name="${prefix}white">
             <color rgba="1.0 1.0 1.0 1.0"/>
         </material>
@@ -84,5 +84,5 @@
         <link name="${prefix}rv2fr_base">
             <visual>
-            <material name="white"/>
+            <material name="${prefix}white"/>
             <origin rpy="0 0 0" xyz="0 0 0"/>
             <geometry>
@@ -102,5 +102,5 @@
         <link name="${prefix}rv2fr_shoulder">
             <visual>
-            <material name="white"/>
+            <material name="${prefix}white"/>
             <origin rpy="0 0 0" xyz="0 0 0"/>
             <geometry>
@@ -120,5 +120,5 @@
         <link name="${prefix}rv2fr_upper_arm">
             <visual>
-            <material name="white"/>
+            <material name="${prefix}white"/>
             <origin rpy="0 0 0" xyz="0 0 0"/>
             <geometry>
@@ -138,5 +138,5 @@
         <link name="${prefix}rv2fr_elbow">
             <visual>
-            <material name="white"/>
+            <material name="${prefix}white"/>
             <origin rpy="0 0 0" xyz="0 0 0"/>
             <geometry>
@@ -156,5 +156,5 @@
         <link name="${prefix}rv2fr_forearm">
             <visual>
-            <material name="white"/>
+            <material name="${prefix}white"/>
             <origin rpy="0 0 0" xyz="0 0 0"/>
             <geometry>
@@ -174,5 +174,5 @@
         <link name="${prefix}rv2fr_wrist">
             <visual>
-            <material name="white"/>
+            <material name="${prefix}white"/>
             <origin rpy="0 0 0" xyz="0 0 0"/>
             <geometry>
@@ -192,5 +192,5 @@
         <link name="${prefix}rv2fr_hand_flange">
             <visual>
-            <material name="white"/>
+            <material name="${prefix}white"/>
             <origin rpy="0 0 0" xyz="0 0 0"/>
             <geometry>

File: melfa_description/urdf/rv4fr/rv4fr_macro.xacro (robot description, xacro)
@@ -19,5 +19,5 @@
         <xacro:property name="wrist_mass" value="0.12190" />
         <xacro:property name="hand_flange_mass" value="0.01879" />
-        <material name="white">
+        <material name="${prefix}white">
             <color rgba="1.0 1.0 1.0 1.0"/>
         </material>
@@ -84,5 +84,5 @@
         <link name="${prefix}rv4fr_base">
             <visual>
-                <material name="white"/>
+                <material name="${prefix}white"/>
                 <origin rpy="0 0 0" xyz="0 0 0"/>
                 <geometry>
@@ -102,5 +102,5 @@
         <link name="${prefix}rv4fr_shoulder">
             <visual>
-            <material name="white"/>
+            <material name="${prefix}white"/>
             <origin rpy="0 0 0" xyz="0 0 0"/>
             <geometry>
@@ -120,5 +120,5 @@
         <link name="${prefix}rv4fr_upper_arm">
             <visual>
-            <material name="white"/>
+            <material name="${prefix}white"/>
             <origin rpy="0 0 0" xyz="0 0 0"/>
             <geometry>
@@ -138,5 +138,5 @@
         <link name="${prefix}rv4fr_elbow">
             <visual>
-            <material name="white"/>
+            <material name="${prefix}white"/>
             <origin rpy="0 0 0" xyz="0 0 0"/>
             <geometry>
@@ -156,5 +156,5 @@
         <link name="${prefix}rv4fr_forearm">
             <visual>
-            <material name="white"/>
+            <material name="${prefix}white"/>
             <origin rpy="0 0 0" xyz="0 0 0"/>
             <geometry>
@@ -174,5 +174,5 @@
         <link name="${prefix}rv4fr_wrist">
             <visual>
-            <material name="white"/>
+            <material name="${prefix}white"/>
             <origin rpy="0 0 0" xyz="0 0 0"/>
             <geometry>
@@ -192,5 +192,5 @@
         <link name="${prefix}rv4fr_hand_flange">
             <visual>
-            <material name="white"/>
+            <material name="${prefix}white"/>
             <origin rpy="0 0 0" xyz="0 0 0"/>
             <geometry>

File: melfa_description/urdf/rv4frl/rv4frl_macro.xacro (robot description, xacro)
@@ -19,5 +19,5 @@
         <xacro:property name="wrist_mass" value="0.12190" />
         <xacro:property name="hand_flange_mass" value="0.01879" />
-        <material name="white">
+        <material name="${prefix}white">
             <color rgba="1.0 1.0 1.0 1.0"/>
         </material>
@@ -83,5 +83,5 @@
         <link name="${prefix}rv4frl_base">
             <visual>
-            <material name="white"/>
+            <material name="${prefix}white"/>
             <origin rpy="0 0 0" xyz="0 0 0"/>
             <geometry>
@@ -101,5 +101,5 @@
         <link name="${prefix}rv4frl_shoulder">
             <visual>
-                <material name="white"/>
+                <material name="${prefix}white"/>
                 <origin rpy="0 0 0" xyz="0 0 0"/>
                 <geometry>
@@ -119,5 +119,5 @@
         <link name="${prefix}rv4frl_upper_arm">
             <visual>
-                <material name="white"/>
+                <material name="${prefix}white"/>
                 <origin rpy="0 0 0" xyz="0 0 0"/>
                 <geometry>
@@ -137,5 +137,5 @@
         <link name="${prefix}rv4frl_elbow">
             <visual>
-                <material name="white"/>
+                <material name="${prefix}white"/>
                 <origin rpy="0 0 0" xyz="0 0 0"/>
                 <geometry>
@@ -155,5 +155,5 @@
         <link name="${prefix}rv4frl_forearm">
             <visual>
-                <material name="white"/>
+                <material name="${prefix}white"/>
                 <origin rpy="0 0 0" xyz="0 0 0"/>
                 <geometry>
@@ -173,5 +173,5 @@
         <link name="${prefix}rv4frl_wrist">
             <visual>
-                <material name="white"/>
+                <material name="${prefix}white"/>
                 <origin rpy="0 0 0" xyz="0 0 0"/>
                 <geometry>
@@ -191,5 +191,5 @@
         <link name="${prefix}rv4frl_hand_flange">
             <visual>
-                <material name="white"/>
+                <material name="${prefix}white"/>
                 <origin rpy="0 0 0" xyz="0 0 0"/>
                 <geometry>

File: melfa_description/urdf/rv5as/rv5as_macro.xacro (robot description, xacro)
@@ -19,5 +19,5 @@
         <xacro:property name="wrist_mass" value="0.12190" />
         <xacro:property name="hand_flange_mass" value="0.01879" />
-        <material name="white">
+        <material name="${prefix}white">
             <color rgba="1.0 1.0 1.0 1.0"/>
         </material>
@@ -84,5 +84,5 @@
         <link name="${prefix}rv5as_base">
             <visual>
-                <material name="white"/>
+                <material name="${prefix}white"/>
                 <origin rpy="0.00 0.00 0.00" xyz="0.00 0.00 0.00"/>
                 <geometry>
@@ -102,5 +102,5 @@
         <link name="${prefix}rv5as_shoulder">
             <visual>
-                <material name="white"/>
+                <material name="${prefix}white"/>
                 <origin rpy="0.00 0.00 0" xyz="0.00 0.00 0.00"/>
                 <geometry>
@@ -120,5 +120,5 @@
         <link name="${prefix}rv5as_upper_arm">
             <visual>
-                <material name="white"/>
+                <material name="${prefix}white"/>
                 <origin rpy="0.00 0.00 0.00" xyz="0.00 0.00 0.00"/>
                 <geometry>
@@ -138,5 +138,5 @@
         <link name="${prefix}rv5as_elbow">
             <visual>
-                <material name="white"/>
+                <material name="${prefix}white"/>
                 <origin rpy="0.00 0.00 0.00" xyz="0.00 0.00 0.00"/>
                 <geometry>
@@ -156,5 +156,5 @@
         <link name="${prefix}rv5as_forearm">
             <visual>
-                <material name="white"/>
+                <material name="${prefix}white"/>
                 <origin rpy="0.00 0.00 0.00" xyz="0.00 0.00 0.00"/>
                 <geometry>
@@ -174,5 +174,5 @@
         <link name="${prefix}rv5as_hand_flange">
             <visual>
-                <material name="white"/>
+                <material name="${prefix}white"/>
                 <origin rpy="0.00 0.00 0.00" xyz="0.00 0.00 0.00"/>
                 <geometry>
@@ -192,5 +192,5 @@
         <link name="${prefix}rv5as_wrist">
             <visual>
-                <material name="white"/>
+                <material name="${prefix}white"/>
                 <origin rpy="0.00 0.00 0.00" xyz="0.00 0.00 0.00"/>
                 <geometry>

File: melfa_description/urdf/rv7frl/rv7frl_macro.xacro (robot description, xacro)
@@ -20,5 +20,5 @@
         <xacro:property name="wrist_mass" value="0.12190" />
         <xacro:property name="hand_flange_mass" value="0.12190" />
-        <material name="white">
+        <material name="${prefix}white">
             <color rgba="1.0 1.0 1.0 1.0"/>
         </material>
@@ -85,5 +85,5 @@
         <link name="${prefix}rv7frl_base">
             <visual>
-                <material name="white"/>
+                <material name="${prefix}white"/>
                 <origin rpy="0 0 0" xyz="0 0 0"/>
                 <geometry>
@@ -103,5 +103,5 @@
         <link name="${prefix}rv7frl_shoulder">
             <visual>
-                <material name="white"/>
+                <material name="${prefix}white"/>
                 <origin rpy="0 0 0" xyz="0 0 0"/>
                 <geometry>
@@ -121,5 +121,5 @@
         <link name="${prefix}rv7frl_upper_arm">
             <visual>
-                <material name="white"/>
+                <material name="${prefix}white"/>
                 <origin rpy="0 0 0" xyz="0 0 0"/>
                 <geometry>
@@ -139,5 +139,5 @@
         <link name="${prefix}rv7frl_elbow">
             <visual>
-                <material name="white"/>
+                <material name="${prefix}white"/>
                 <origin rpy="0 0 0" xyz="0 0 0"/>
                 <geometry>
@@ -157,5 +157,5 @@
         <link name="${prefix}rv7frl_forearm">
             <visual>
-                <material name="white"/>
+                <material name="${prefix}white"/>
                 <origin rpy="0 0 0" xyz="0 0 0"/>
                 <geometry>
@@ -175,5 +175,5 @@
         <link name="${prefix}rv7frl_wrist">
             <visual>
-                <material name="white"/>
+                <material name="${prefix}white"/>
                 <origin rpy="0 0 0" xyz="0 0 0"/>
                 <geometry>
@@ -193,5 +193,5 @@
         <link name="${prefix}rv7frl_hand_flange">
             <visual>
-                <material name="white"/>
+                <material name="${prefix}white"/>
                 <origin rpy="0 0 0" xyz="0 0 0"/>
                 <geometry>

File: melfa_description/urdf/rv80fr/rv80fr_macro.xacro (robot description, xacro)
@@ -19,5 +19,5 @@
         <xacro:property name="wrist_mass" value="0.12190" />
         <xacro:property name="hand_flange_mass" value="0.12190" />
-        <material name="white">
+        <material name="${prefix}white">
             <color rgba="1.0 1.0 1.0 1.0"/>
         </material>
@@ -84,5 +84,5 @@
         <link name="${prefix}rv80fr_base">
             <visual>
-                <material name="white"/>
+                <material name="${prefix}white"/>
                 <origin rpy="0 0 0" xyz="0 0 0"/>
                 <geometry>
@@ -102,5 +102,5 @@
         <link name="${prefix}rv80fr_shoulder">
             <visual>
-                <material name="white"/>
+                <material name="${prefix}white"/>
                 <origin rpy="0 0 0" xyz="0 0 0"/>
                 <geometry>
@@ -120,5 +120,5 @@
         <link name="${prefix}rv80fr_upper_arm">
             <visual>
-                <material name="white"/>
+                <material name="${prefix}white"/>
                 <origin rpy="0 0 0" xyz="0 0 0"/>
                 <geometry>
@@ -138,5 +138,5 @@
         <link name="${prefix}rv80fr_elbow">
             <visual>
-                <material name="white"/>
+                <material name="${prefix}white"/>
                 <origin rpy="0 0 0" xyz="0 0 0"/>
                 <geometry>
@@ -156,5 +156,5 @@
         <link name="${prefix}rv80fr_forearm">
             <visual>
-                <material name="white"/>
+                <material name="${prefix}white"/>
                 <origin rpy="0 0 0" xyz="0 0 0"/>
                 <geometry>
@@ -174,5 +174,5 @@
         <link name="${prefix}rv80fr_wrist">
             <visual>
-                <material name="white"/>
+                <material name="${prefix}white"/>
                 <origin rpy="0 0 0" xyz="0 0 0"/>
                 <geometry>
@@ -192,5 +192,5 @@
         <link name="${prefix}rv80fr_hand_flange">
             <visual>
-                <material name="white"/>
+                <material name="${prefix}white"/>
                 <origin rpy="0 0 0" xyz="0 0 0"/>
                 <geometry>

File: melfa_description/urdf/rv8crl/rv8crl_macro.xacro (robot description, xacro)
@@ -19,5 +19,5 @@
         <xacro:property name="wrist_mass" value="0.12190" />
         <xacro:property name="hand_flange_mass" value="0.01879" />
-        <material name="white">
+        <material name="${prefix}white">
             <color rgba="1.0 1.0 1.0 1.0"/>
         </material>
@@ -84,5 +84,5 @@
         <link name="${prefix}rv8crl_base">
             <visual>
-            <material name="white"/>
+            <material name="${prefix}white"/>
             <origin rpy="0 0 0" xyz="0 0 0"/>
             <geometry>
@@ -102,5 +102,5 @@
         <link name="${prefix}rv8crl_shoulder">
             <visual>
-            <material name="white"/>
+            <material name="${prefix}white"/>
             <origin rpy="0 0 0" xyz="0 0 0"/>
             <geometry>
@@ -120,5 +120,5 @@
         <link name="${prefix}rv8crl_upper_arm">
             <visual>
-            <material name="white"/>
+            <material name="${prefix}white"/>
             <origin rpy="0 0 0" xyz="0 0 0"/>
             <geometry>
@@ -138,5 +138,5 @@
         <link name="${prefix}rv8crl_elbow">
             <visual>
-            <material name="white"/>
+            <material name="${prefix}white"/>
             <origin rpy="0 0 0" xyz="0 0 0"/>
             <geometry>
@@ -156,5 +156,5 @@
         <link name="${prefix}rv8crl_forearm">
             <visual>
-            <material name="white"/>
+            <material name="${prefix}white"/>
             <origin rpy="0 0 0" xyz="0 0 0"/>
             <geometry>
@@ -174,5 +174,5 @@
         <link name="${prefix}rv8crl_wrist">
             <visual>
-            <material name="white"/>
+            <material name="${prefix}white"/>
             <origin rpy="0 0 0" xyz="0 0 0"/>
             <geometry>
@@ -192,5 +192,5 @@
         <link name="${prefix}rv8crl_hand_flange">
             <visual>
-            <material name="white"/>
+            <material name="${prefix}white"/>
             <origin rpy="0 0 0" xyz="0 0 0"/>
             <geometry>
